File: my_design/Slimme_meter_Sim/SCH_1_USB_5volt_sch.kicad_sch (KiCad schematic)
At the start: 29 parts, among them CN1 S2B-PH-SM4-TB, SW1 MSK12C02, U1 USBLC6-2SC6-ES, U2 BQ25185DLHR, U3 TPS61023DRLR

Commit message: Add sheet-2 power/MCU schematic progress and document P1 opto domains.
Captures TPS26625, SY8088 3V3, ESP32-C3, RJ12 placement, and README guidance that Request/Data optos keep UART on 3.3 V while pin 5 stays open-collector on the 5 V P1 side.

Co-authored-by: Cursor <cursoragent@cursor.com>
Changed lines of the file:
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@@
 	(wire
 		(pts
+			(xy 332.74 77.47) (xy 332.74 76.2)
+		)
+		(stroke
+			(width 0)
+			(type default)
+		)
+	)
+	(wire
+		(pts
 			(xy 234.95 64.77) (xy 240.03 64.77)
 		)
@@
 	(wire
 		(pts
+			(xy 332.74 76.2) (xy 334.01 76.2)
+		)
+		(stroke
+			(width 0)
+			(type default)
+		)
+	)
+	(wire
+		(pts
 			(xy 87.63 50.8) (xy 87.63 36.83)
 		)
@@
 		)
 	)
+	(hierarchical_label "+5V"
+		(shape bidirectional)
+		(at 332.74 72.39 0)
+		(effects
+			(font
+				(size 1.27 1.27)
+			)
+			(justify left)
+		)
+	)
+	(hierarchical_label "GND1"
+		(shape bidirectional)
+		(at 334.01 76.2 0)
+		(effects
+			(font
+				(size 1.27 1.27)
+			)
+			(justify left)
+		)
+	)
 	(symbol
 		(lib_id "power:VCC")
@@
 	(symbol
 		(lib_id "power:GND1")
+		(at 332.74 77.47 0)
+		(unit 1)
+		(exclude_from_sim no)
+		(in_bom yes)
+		(on_board yes)
+		(dnp no)
+		(fields_autoplaced yes)
+		(property "Reference" "#PWR041"
+			(at 332.74 83.82 0)
+			(effects
+				(font
+					(size 1.27 1.27)
+				)
+				(hide yes)
+			)
+		)
+		(property "Value" "GND1"
+			(at 332.74 82.55 0)
+			(effects
+				(font
+					(size 1.27 1.27)
+				)
+			)
+		)
+		(property "Footprint" ""
+			(at 332.74 77.47 0)
+			(effects
+				(font
+					(size 1.27 1.27)
+				)
+				(hide yes)
+			)
+		)
+		(property "Datasheet" ""
+			(at 332.74 77.47 0)
+			(effects
+				(font
+					(size 1.27 1.27)
+				)
+				(hide yes)
+			)
+		)
+		(property "Description" "Power symbol creates a global label with name \"GND1\" , ground"
+			(at 332.74 77.47 0)
+			(effects
+				(font
+					(size 1.27 1.27)
+				)
+				(hide yes)
+			)
+		)
+		(pin "1"
+		)
+		(instances
+			(project "Slimme_meter_Sim"
+				(path "/d59de98b-abe3-4329-b084-e6d28a71ec22/5e636416-256f-40d4-bd94-a88f282663f2"
+					(reference "#PWR041")
+					(unit 1)
+				)
+			)
+		)
+	)
+	(symbol
+		(lib_id "power:GND1")
 		(at 151.13 153.67 0)
 		(unit 1)
@@
 					(unit 1)
 				)
+			)
+		)
+	)
+	(symbol
+		(lib_id "power:+5V")
+		(at 332.74 72.39 0)
+		(unit 1)
+		(exclude_from_sim no)
+		(in_bom yes)
+		(on_board yes)
+		(dnp no)
+		(fields_autoplaced yes)
+		(property "Reference" "#PWR040"
+			(at 332.74 76.2 0)
+			(effects
+				(font
+					(size 1.27 1.27)
+				)
+				(hide yes)
+			)
+		)
+		(property "Value" "+5V"
+			(at 332.74 67.31 0)
+			(effects
+				(font
+					(size 1.27 1.27)
+				)
+			)
+		)
+		(property "Footprint" ""
+			(at 332.74 72.39 0)
+			(effects
+				(font
+					(size 1.27 1.27)
+				)
+				(hide yes)
+			)
+		)
+		(property "Datasheet" ""
+			(at 332.74 72.39 0)
+			(effects
+				(font
+					(size 1.27 1.27)
+				)
+				(hide yes)
+			)
+		)
+		(property "Description" "Power symbol creates a global label with name \"+5V\""
+			(at 332.74 72.39 0)
+			(effects
+				(font
+					(size 1.27 1.27)
+				)
+				(hide yes)
+			)
+		)
+		(pin "1"
+		)
+		(instances
+			(project "Slimme_meter_Sim"
+				(path "/d59de98b-abe3-4329-b084-e6d28a71ec22/5e636416-256f-40d4-bd94-a88f282663f2"
+					(reference "#PWR040")
+					(unit 1)
+				)

Commit message: Save KiCad schematic/PCB progress and park Pi next-step ideas.
Document assembly (stencil + hot air) and the dual-domain Pi brain option so the ESP32 path can be resumed cleanly tomorrow.

Co-authored-by: Cursor <cursoragent@cursor.com>
Parts:
- added C20, C21, C23: CL05B104KO5NNNC, EasyEDA:C0402, symbol EasyEDA:CL05B104KO5NNNC
- added C22: FS31X226M160EPG, EasyEDA:C1206, symbol EasyEDA:FS31X226M160EPG
Connections:
- net +5V: now also C23.1
- net GND1: now also C20.1, C21.2, C22.2, C23.2
- net VCC: now also C21.1, C22.1
- net at C1.2, D1.1 (C), U2.10 (IN): now also C20.2
Other:
- moved on the sheet: D1

Commit message: Save Slimme_meter_Sim KiCad progress: PCB/schematic, footprints, and firmware pin map.
Co-authored-by: Cursor <cursoragent@cursor.com>
Parts:
- removed R3, R4: AR02BTC5101, EasyEDA:R0402, symbol EasyEDA:AR02BTC5101
- removed R9: AR02BTC1002, EasyEDA:R0402, symbol EasyEDA:AR02BTC1002
- added BT1, BT2: BH-18650-B1BA002, EasyEDA:BATTERY-SMD_18650-1S-L77.1-W20.7-1, symbol EasyEDA:BH-18650-B1BA002
- added Batt_power_on_SW1, USB_power_on_SW1: ST-0-102-C04-N008-RS, EasyEDA:SW-TH_ST-0-102-C04-N008-RS, symbol EasyEDA:ST-0-102-C04-N008-RS
- added C31: CL05B104KO5NNNC, EasyEDA:C0402, symbol EasyEDA:CL05B104KO5NNNC
- added CN2: S2B-PH-SM4-TB, EasyEDA:CONN-SMD_P2.00_S2B-PH-SM4-TB-LF-SN, symbol EasyEDA:S2B-PH-SM4-TB
- added R3, R4, R47: RC0603JR-071KL, EasyEDA:R0603, symbol EasyEDA:RC0603JR-071KL
- added R39, R40: 0402WGF1003TCE, EasyEDA:R0402, symbol EasyEDA:0402WGF1003TCE
Connections:
- net +5V: now also R4.2
- net 5V_usb: now also USB_power_on_SW1.3; no longer D1.2 (A)
- net GND1: now also BT1.1, BT2.1, Batt_power_on_SW1.4, C31.2, CN2.2, CN2.3, CN2.4, R40.2, USB_power_on_SW1.4
- net VBATT: now also Batt_power_on_SW1.2, R39.1; no longer CN1.1
- net stat1: now also R3.1
- net stat2: now also R47.2
- net at LED3_orange1.1 (K): now also R47.1
- net at LED1_red1.2 (K): now also R3.2
- net at LED2.2 (A): now also R4.1
- new net 5V_usb_1: D1.2 (A), USB_power_on_SW1.2
- new net GPIO4_Battery: C31.1, R39.2, R40.1
- new net V_batt_port: BT1.2, BT2.2, Batt_power_on_SW1.3, CN1.1, CN2.1

Commit message: Save production-ready Slimme_meter_Sim Gerbers, JLCPCB BOM/CPL, and finished PCB.
Co-authored-by: Cursor <cursoragent@cursor.com>
Parts:
- removed BT2: BH-18650-B1BA002, EasyEDA:BATTERY-SMD_18650-1S-L77.1-W20.7-1, symbol EasyEDA:BH-18650-B1BA002
Other:
- moved on the sheet: BT1, Batt_power_on_SW1, C31, CN1, CN2, R39, R40
