File: my_design/Slimme_meter_Sim/SCH_2_power_supplies.kicad_sch (KiCad schematic)
At the start: 49 parts, among them U4 TPS26625DRCR, U5 C1206C105K3RACAUTO, U6 SY8088AAC, U7 ESP32-C3-MINI-1-H4X

Commit message: Save KiCad schematic/PCB progress and park Pi next-step ideas.
Document assembly (stencil + hot air) and the dual-domain Pi brain option so the ESP32 path can be resumed cleanly tomorrow.

Co-authored-by: Cursor <cursoragent@cursor.com>
Parts:
- removed H2 (x2): ~, PCM_fab:MountingHole_M2, symbol PCM_fab:MountingHole_M2
- added C19, C24, C25: CL05B104KO5NNNC, EasyEDA:C0402, symbol EasyEDA:CL05B104KO5NNNC
- added H10, H11, H2, H5, H6, H7, H8, H9: ~, PCM_fab:MountingHole_M2, symbol PCM_fab:MountingHole_M2
- added R29, R32, R33: AR02BTC1002, EasyEDA:R0402, symbol EasyEDA:AR02BTC1002
- added R30: MCS04020C2200FE000, EasyEDA:R0402, symbol EasyEDA:MCS04020C2200FE000
- added R31: 25121WJ0331T4E, EasyEDA:R2512, symbol EasyEDA:25121WJ0331T4E
- added SW2: KMR231GLFS, EasyEDA:KEY-SMD_KMR2XXGXXX, symbol EasyEDA:KMR231GLFS
- added U8, U9: 6N137S_C20612601, EasyEDA:SOP-8_L9.7-W6.5-P2.54-LS10.3-BL, symbol EasyEDA:6N137S_C20612601
- renumbered GND to GND1
Connections:
- net +3V3: now also R29.2, R33.1
- net +5V: now also C19.2, C24.1, C25.1, R32.1, U8.7 (VB), U8.8 (VCC), U9.7 (VB), U9.8 (VCC); no longer C12.2, U6.1 (EN)
- net GND1: now also C19.1, C24.2, C25.2, SW2.1, SW2.2, SW2.5, U8.1 (N/C), U8.3 (CAT), U8.4 (N/C), U8.5 (GND), U9.1 (N/C), U9.3 (CAT), U9.4 (N/C), U9.5 (GND)
- net RJ12_Tx_pin5: now also U8.6 (VO)
- net ESP32_Sw: now reaches U7.18 (IO4)
- net ESP32_Sw: now also R29.1, SW2.3, SW2.4
- net ESP32_enable: now reaches U7.19 (IO5)
- net ESP32_enable: now also R33.2, U9.6 (VO)
- net USB_D-: now reaches U7.26 (IO18)
- net USB_D+: now reaches U7.27 (IO19)
- net ESP32_TX: now reaches U7.31 (TXD0)
- net ESP32_TX: now also R30.1
- net RJ12_Enable renamed RJ12_pin2
- net RJ12_pin2: now also R31.1
- new net: C12.2, R32.2, U6.1 (EN)
- new net: R31.2, U9.2 (AN)
- new net: R30.2, U8.2 (AN)

Commit message: Save Slimme_meter_Sim KiCad progress: PCB/schematic, footprints, and firmware pin map.
Co-authored-by: Cursor <cursoragent@cursor.com>
Parts:
- removed H1: DS1023-2*5SF11, EasyEDA:HDR-TH_10P-P2.54-V-F-R2-C5-S2.54, symbol EasyEDA:DS1023-2*5SF11
- removed H10, H11: ~, PCM_fab:MountingHole_M2, symbol PCM_fab:MountingHole_M2
- removed R20: AR03FTC2672, EasyEDA:R0603, symbol EasyEDA:AR03FTC2672
- removed SW2: KMR231GLFS, EasyEDA:KEY-SMD_KMR2XXGXXX, symbol EasyEDA:KMR231GLFS
- removed TP2: RH-5002, EasyEDA:TESTPOINT-TH_BD2.5-D1.2_RH-5002, symbol EasyEDA:RH-5002
- added C26: CL05A105KA5NQNC, EasyEDA:C0402, symbol EasyEDA:CL05A105KA5NQNC
- added C27, C30: FS31X226M160EPG, EasyEDA:C1206, symbol EasyEDA:FS31X226M160EPG
- added C28, C29: CL05B104KO5NNNC, EasyEDA:C0402, symbol EasyEDA:CL05B104KO5NNNC
- added Card1: DM3AT-SF-PEJM5, EasyEDA:SD-SMD_DM3AT-SF-PEJM5, symbol EasyEDA:DM3AT-SF-PEJM5
- added D5: RCLAMP0524P_C907837, EasyEDA:DFN2510-10_L2.5-W1.0-P0.50-BL, symbol EasyEDA:RCLAMP0524P_C907837
- added R34, R35, R36, R38, R41, R42, R43, R44, R45, R46: AR02BTC1002, EasyEDA:R0402, symbol EasyEDA:AR02BTC1002
- added R37: 25121WJ0331T4E, EasyEDA:R2512, symbol EasyEDA:25121WJ0331T4E
- added R9: RC0603JR-071KL, EasyEDA:R0603, symbol EasyEDA:RC0603JR-071KL
- added SW2, SW3: TS665CJ, EasyEDA:SW-TH_4P-L6.0-W6.0-P4.50-LS6.5, symbol EasyEDA:TS665CJ
- added SW4: SK-1500-L1?, EasyEDA:SW-SMD_6P-P1.50_L2.7-W11.2, symbol EasyEDA:SK-1500-L1?
- added U10: 6N137S_C20612601, EasyEDA:SOP-8_L9.7-W6.5-P2.54-LS10.3-BL, symbol EasyEDA:6N137S_C20612601
- added U11, U12, U13: C1206C105K3RACAUTO, EasyEDA:C1206, symbol EasyEDA:C1206C105K3RACAUTO
- H2, H3, H4, H5, H6, H7, H8, H9: footprint PCM_fab:MountingHole_M2 -> MountingHole:MountingHole_3.2mm_M3; symbol PCM_fab:MountingHole_M2 -> PCM_SL_Mechanical:MountingHole_M3; now in the parts list
- renumbered TP1 to RJ12_5V1
Connections:
- net +3V3: now also C27.2, C29.2, C30.2, Card1.4 (VDD), R34.2, R35.1, R36.1, R38.1, R41.1, R42.1, R43.1, R44.1, R45.1, R46.1
- net +5V: now also C28.1, R37.1, U10.7 (VB), U10.8 (VCC), U11.1, U12.1, U13.1
- net ESP32_Sw: now also C17.2, R26.2, U7.8 (EN), SW2.3 (C), SW2.4 (D); no longer U7.18 (IO4)
- net GND1: now also C26.1, C27.1, C28.2, C29.1, C30.1, Card1.10, Card1.12, Card1.13, Card1.14, Card1.6 (VSS), Card1.9 (SW_B), D5.3 (GND), D5.8 (GND), SW2.1 (A), SW2.2 (B), SW3.1 (A), SW3.2 (B), SW4.10, SW4.7, SW4.8, SW4.9, U10.1 (N/C), U10.4 (N/C), U10.5 (GND), U11.2, U12.2, U13.2
- net RJ12_5V: now also R9.2
- net at R14.2: now also SW4.6
- net at U4.7 (ILIM): now also SW4.3, SW4.4
- net at R15.2: now also SW4.5
- net at R16.2: now also SW4.2
- net at R17.1: now also SW4.1
- net GPIO0_SCK: now reaches U7.12 (IO0)
- net GPIO0_SCK: now also Card1.5 (CLK), D5.4 (I/O3), D5.7 (NC), R43.2
- net GPIO1_MOSI_CMD: now reaches U7.13 (IO1)
- net GPIO1_MOSI_CMD: now also Card1.3 (CMD), D5.2 (I/O2), D5.9 (NC), R42.2
- net GPIO6_CS: now reaches U7.20 (IO6)
- net GPIO6_CS: now also Card1.2 (CD/DAT3), D5.1 (I/O1), D5.10 (NC), R41.2
- net SD_CD_SW_A: now reaches U7.21 (IO7)
- net SD_CD_SW_A: now also Card1.11 (SW_A), R45.2
- net ESP32_Sw_GPIO9: now reaches U7.23 (IO9)
- net ESP32_Sw_GPIO9: now also C26.2, R34.1, R35.2, SW3.3 (C), SW3.4 (D)
- net ESP32_FLT_Efuse: now reaches U7.30 (RXD0)
- net ESP32_FLT_Efuse: now also R38.2, U10.6 (VO)
- net GPIO3_MISO: now reaches U7.6 (IO3)
- net GPIO3_MISO: now also Card1.7 (DAT0), D5.5 (I/O4), D5.6 (NC), R44.2
- net at LED1.2 (A): now also R9.1
- new net: Card1.8 (DAT1), R46.2
- new net: R37.2, U10.2 (AN)
- new net: Card1.1 (DAT2), R36.2
- new net Efuse_FLT: U10.3 (CAT)
- new net GPIO4_Battery: U7.18 (IO4)
Other:
- moved on the sheet: R14, R22, R29

Commit message: Save production-ready Slimme_meter_Sim Gerbers, JLCPCB BOM/CPL, and finished PCB.
Co-authored-by: Cursor <cursoragent@cursor.com>
Parts:
- removed C26: CL05A105KA5NQNC, EasyEDA:C0402, symbol EasyEDA:CL05A105KA5NQNC
- removed R30: MCS04020C2200FE000, EasyEDA:R0402, symbol EasyEDA:MCS04020C2200FE000
- removed R31, R37: 25121WJ0331T4E, EasyEDA:R2512, symbol EasyEDA:25121WJ0331T4E
- added H1, H10, H11, H12: ~, PCM_fab:MountingHole_M2, symbol PCM_fab:MountingHole_M2
- added R20, R30: ERJP03F3300V, EasyEDA:R0603, symbol EasyEDA:ERJP03F3300V
- added R37: 0603WAF2200T5E, EasyEDA:R0603, symbol EasyEDA:0603WAF2200T5E
- H2, H3, H4, H5, H6, H7, H8, H9: now left out of the parts list
- R17: Manufacturer (none) -> HRC0603F2673ENTN
Connections:
- net +5V: now also R20.1
- net ESP32_TX: now also R37.1
- net Efuse_FLT: now also R21.2, U4.9 (~{FLT})
- net RJ12_pin2: now also R30.1
- net at U9.2 (AN): now also R30.2
- net at U10.2 (AN): now also R20.2
- net at U8.2 (AN): now also R37.2
Other:
- moved on the sheet: C24, C25, H2, H3, H4, H5, H6, H7, H8, H9, R29, R33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
