File: my_design/Slimme_meter_Sim -big-modular/SCH_1_USB_5volt_sch.kicad_sch (KiCad schematic)
At the start: 40 parts, among them CN1 S2B-PH-SM4-TB, CN2 S2B-PH-SM4-TB, SW1 MSK12C02, U1 USBLC6-2SC6-ES, U2 BQ25185DLHR, U3 TPS61023DRLR

Commit message: Lock big-modular plan on DevKitC WROOM-2 with dual eFuse and safe 5V powering.
Document diode/switch power rules, USB-C/SD breakouts, N32R16V MCU module, and continue KiCad power sheets for the hand-build carrier.

Co-authored-by: Cursor <cursoragent@cursor.com>
Parts:
- added USB_c1: PINHD_1x6_Female, Connector_PinSocket_2.54mm:PinSocket_1x06_P2.54mm_Vertical, symbol PCM_SL_Pin_Headers:PINHD_1x6_Female
Connections:
- net 5V_usb: now also USB_c1.2
- net GND1: now also USB_c1.1
Other:
- moved on the sheet: BT1, Batt_power_on_SW1, C1, C2, C20, C21, C22, C23, C3, C31, C4, C5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

Commit message: Checkpoint big-modular KiCad and FP6276B tooling before deeper power modularization.
Save DevKitC reference assets, USB-C breakout zip, boost datasheet/designer, and current schematic/PCB/library progress on the hand-build path.

Co-authored-by: Cursor <cursoragent@cursor.com>
Parts:
- removed R1, R2: AR02BTC5101, EasyEDA:R0402, symbol EasyEDA:AR02BTC5101
- removed U1: USBLC6-2SC6-ES, EasyEDA:SOT-23-6_L2.9-W1.6-P0.95-LS2.8-BR, symbol EasyEDA:USBLC6-2SC6-ES
- removed U3: TPS61023DRLR, EasyEDA:SOT-563_L1.6-W1.2-P0.50-LS1.6-BR, symbol EasyEDA:TPS61023DRLR
- removed USBC1: TYPE-C-31-M-12, foot:USB-C_SMD-TYPE-C-31-M-12_1, symbol EasyEDA:TYPE-C-31-M-12
- removed USB_c1: PINHD_1x6_Female, Connector_PinSocket_2.54mm:PinSocket_1x06_P2.54mm_Vertical, symbol PCM_SL_Pin_Headers:PINHD_1x6_Female
- added C13: FS31X226M160EPG, EasyEDA:C1206, symbol EasyEDA:FS31X226M160EPG
- added J5: PINHD_1x8_Female, Connector_PinSocket_2.54mm:PinSocket_1x08_P2.54mm_Vertical, symbol PCM_SL_Pin_Headers:PINHD_1x8_Female
- added R1: FRC1206J104 TS, EasyEDA:R1206, symbol EasyEDA:FRC1206J104TS
- added U1: TPS61022RWUR, EasyEDA:VQFN-7_L2.0-W2.0-P0.55-TL_RWU, symbol EasyEDA:TPS61022RWUR
- C20, C21, C23, C31: value CL05B104KO5NNNC -> TCC1206M3L104J500FT; footprint EasyEDA:C0402 -> EasyEDA:C1206; symbol EasyEDA:CL05B104KO5NNNC -> EasyEDA:TCC1206M3L104J500FT; LCSC Part C1525 -> C359189; MPN CL05B104KO5NNNC -> TCC1206M3L104J500FT; Manufacturer SAMSUNG(三星) -> CCTC(三环)
- R10, R12, R39, R40: value 0402WGF1003TCE -> FRC1206J104 TS; footprint EasyEDA:R0402 -> EasyEDA:R1206; symbol EasyEDA:0402WGF1003TCE -> EasyEDA:FRC1206J104TS; LCSC Part C25741 -> C2907421; MPN 0402WGF1003TCE -> FRC1206J104 TS; Manufacturer UNI-ROYAL(厚声) -> FOJAN(富捷)
- R11: value FRC0402F7323TS -> RC1206FR-07732KL; footprint EasyEDA:R0402 -> EasyEDA:R1206; symbol EasyEDA:FRC0402F7323TS -> EasyEDA:RC1206FR-07732KL; LCSC Part C5159692 -> C488960; MPN FRC0402F7323TS -> RC1206FR-07732KL; Manufacturer FOJAN(富捷) -> YAGEO(国巨)
- R3, R4, R47: value RC0603JR-071KL -> FRC1206F1R30TS; footprint EasyEDA:R0603 -> EasyEDA:R1206; symbol EasyEDA:RC0603JR-071KL -> EasyEDA:FRC1206F1R30TS; LCSC Part C14676 -> C2907365; MPN RC0603JR-071KL -> FRC1206F1R30TS; Manufacturer YAGEO(国巨) -> FOJAN(富捷)
- R5: value AR02BTC1002 -> 1206W4F1002T5E; footprint EasyEDA:R0402 -> EasyEDA:R1206; symbol EasyEDA:AR02BTC1002 -> EasyEDA:1206W4F1002T5E; LCSC Part C317926 -> C17902; MPN AR02BTC1002 -> 1206W4F1002T5E; Manufacturer Viking(光颉) -> UNI-ROYAL(厚声)
Connections:
- net +5V: now also C23.2, U1.3 (VOUT); no longer C23.1
- net 5V_usb: now also J5.2
- net GND1: now also C20.2, C21.1, C23.1, C31.1, C13.2, J5.1, U1.1 (GND); no longer C20.1, C21.2, C23.2, C31.2
- net GPIO4_Battery: now also C31.2; no longer C31.1
- net VCC: now also C21.2, C13.1, R1.2, U1.7 (VIN); no longer C21.1
- net FB_booster: now reaches R11.1, R12.2
- net FB_booster: now also U1.4 (FB)
- net at C1.2, D1.1 (C), U2.10 (IN): now also C20.1; no longer C20.2
- net at R10.1: now also U1.5 (EN)
- net SW_booster: now reaches L1.2
- net SW_booster: now also U1.2 (SW)
- new net: R1.1, U1.6 (MODE)
- no-connect marks 3 -> 1
Other:
- moved on the sheet: BT1, Batt_power_on_SW1, C21, C22, C23, C31, C4, C5, C6, CN1, CN2, L1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
