File: my_design/Slimme_meter_Sim -big-modular/SCH_2_power_supplies.kicad_sch (KiCad schematic)
At the start: 89 parts, among them SW2 TS665CJ, SW3 TS665CJ, SW4 SK-1500-L1?, U10 6N137S_C20612601, U11 C1206C105K3RACAUTO, U12 C1206C105K3RACAUTO, U13 C1206C105K3RACAUTO, U4 TPS26625DRCR, U5 C1206C105K3RACAUTO, U6 SY8088AAC, U7 ESP32-C3-MINI-1-H4X, U8 6N137S_C20612601, U9 6N137S_C20612601

Commit message: Lock big-modular plan on DevKitC WROOM-2 with dual eFuse and safe 5V powering.
Document diode/switch power rules, USB-C/SD breakouts, N32R16V MCU module, and continue KiCad power sheets for the hand-build carrier.

Co-authored-by: Cursor <cursoragent@cursor.com>
Parts:
- added J1, J3: PINHD_1x20_Female, Connector_PinSocket_2.54mm:PinSocket_1x20_P2.54mm_Vertical, symbol PCM_SL_Pin_Headers:PINHD_1x20_Female
- added J2, J4: PINHD_1x2_Female, Connector_PinSocket_2.54mm:PinSocket_1x02_P2.54mm_Vertical, symbol PCM_SL_Pin_Headers:PINHD_1x2_Female
- added SD_card_254: PINHD_1x8_Female, Connector_PinSocket_2.54mm:PinSocket_1x08_P2.54mm_Vertical, symbol PCM_SL_Pin_Headers:PINHD_1x8_Female
- added U14: TPS2553DBVR, EasyEDA:SOT-23-6_L2.9-W1.6-P0.95-LS2.8-BR, symbol EasyEDA:TPS2553DBVR
- added U15: ESP32-S3-DevKitC, PCM_Espressif:ESP32-S3-DevKitC, symbol PCM_Espressif:ESP32-S3-DevKitC
Connections:
- new net: U15.1 (3V3), U15.2 (3V3)
- new net: U15.22 (GND), U15.23 (GND), U15.24 (GND), U15.44 (GND)
- new net 3v: SD_card_254.7
- new net 5V: SD_card_254.8
- new net CD: SD_card_254.1
- new net CLK: SD_card_254.5
- new net DI: SD_card_254.3
- new net DO: SD_card_254.4
- new net GND: SD_card_254.6
- new net cs: SD_card_254.2
Other:
- moved on the sheet: C15, C16, C17, C18, C27, C29, C30, Card1, D4, D5, LED3, R25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

Commit message: Checkpoint big-modular KiCad and FP6276B tooling before deeper power modularization.
Save DevKitC reference assets, USB-C breakout zip, boost datasheet/designer, and current schematic/PCB/library progress on the hand-build path.

Co-authored-by: Cursor <cursoragent@cursor.com>
Parts:
- removed 3v3: RH-5117, EasyEDA:TESTPOINT-TH_BD3.2-D1.6, symbol EasyEDA:RH-5117
- removed C11, C13, C14, C16, C27: FS31X226M160EPG, EasyEDA:C1206, symbol EasyEDA:FS31X226M160EPG
- removed C12, C17: CL05A105KA5NQNC, EasyEDA:C0402, symbol EasyEDA:CL05A105KA5NQNC
- removed C15, C18: CL05B104KO5NNNC, EasyEDA:C0402, symbol EasyEDA:CL05B104KO5NNNC
- removed Card1: DM3AT-SF-PEJM5, EasyEDA:SD-SMD_DM3AT-SF-PEJM5, symbol EasyEDA:DM3AT-SF-PEJM5
- removed D4: B5819W_C8598, EasyEDA:SOD-123_L2.7-W1.6-LS3.7-RD-1, symbol EasyEDA:B5819W_C8598
- removed D5: RCLAMP0524P_C907837, EasyEDA:DFN2510-10_L2.5-W1.0-P0.50-BL, symbol EasyEDA:RCLAMP0524P_C907837
- removed GND1: RH-5002, EasyEDA:TESTPOINT-TH_BD2.5-D1.2_RH-5002, symbol EasyEDA:RH-5002
- removed L2: MDTA32251B-2R2M, EasyEDA:IND-SMD_L3.2-W2.5-BRL3225T100M, symbol EasyEDA:MDTA32251B-2R2M
- removed LED3: DY-S505016/RGBC/6812F-NL-1T, EasyEDA:LED-SMD_4P-L5.0-W5.0-BR, symbol EasyEDA:DY-S505016_RGBC_6812F-NL-1T
- removed R23: RT0402FRE07309RL, EasyEDA:R0402, symbol EasyEDA:RT0402FRE07309RL
- removed R24: SCR0402F68R1, EasyEDA:R0402, symbol EasyEDA:SCR0402F68R1
- removed R25, R26, R27, R29, R32, R34, R35, R36, R41, R42, R43, R44, R45, R46: AR02BTC1002, EasyEDA:R0402, symbol EasyEDA:AR02BTC1002
- removed R28: 0402WGF3300TCE, EasyEDA:R0402, symbol EasyEDA:0402WGF3300TCE
- removed SW2, SW3: TS665CJ, EasyEDA:SW-TH_4P-L6.0-W6.0-P4.50-LS6.5, symbol EasyEDA:TS665CJ
- removed U6: SY8088AAC, EasyEDA:SOT-23-5_L3.0-W1.7-P0.95-LS2.8-BR, symbol EasyEDA:SY8088AAC
- removed U7: ESP32-C3-MINI-1-H4X, EasyEDA:WIFIM-SMD_ESP32-C3-MINI-1, symbol EasyEDA:ESP32-C3-MINI-1-H4X
- added C11: TCC1206M3L104J500FT, EasyEDA:C1206, symbol EasyEDA:TCC1206M3L104J500FT
- added C12: FS31X226M160EPG, EasyEDA:C1206, symbol EasyEDA:FS31X226M160EPG
- C19, C24, C25, C28, C29: value CL05B104KO5NNNC -> TCC1206M3L104J500FT; footprint EasyEDA:C0402 -> EasyEDA:C1206; symbol EasyEDA:CL05B104KO5NNNC -> EasyEDA:TCC1206M3L104J500FT; LCSC Part C1525 -> C359189; MPN CL05B104KO5NNNC -> TCC1206M3L104J500FT; Manufacturer SAMSUNG(三星) -> CCTC(三环)
- C8: value GRM188R71H223KA01D -> GRM3195C1H223JA01D; footprint EasyEDA:C0603 -> EasyEDA:C1206; symbol EasyEDA:GRM188R71H223KA01D -> EasyEDA:GRM3195C1H223JA01D; LCSC Part C77056 -> C97929; MPN GRM188R71H223KA01D -> GRM3195C1H223JA01D
- R13: value CR0603-FX-3012ELF -> FRC1206F3012TS; footprint EasyEDA:R0603 -> EasyEDA:R1206; symbol EasyEDA:CR0603-FX-3012ELF -> EasyEDA:FRC1206F3012TS; LCSC Part C203506 -> C48533691; MPN CR0603-FX-3012ELF -> FRC1206F3012TS; Manufacturer BOURNS -> FOJAN(富捷)
- R18: value CR0603-FX-3742ELF -> WR12X3742FTL; footprint EasyEDA:R0603 -> EasyEDA:R1206; symbol EasyEDA:CR0603-FX-3742ELF -> EasyEDA:WR12X3742FTL; LCSC Part C203565 -> C908492; MPN CR0603-FX-3742ELF -> WR12X3742FTL; Manufacturer BOURNS -> Walsin(华新科)
- R19: value RS-03K1583FT -> CL1206FN158KPS; footprint EasyEDA:R0603 -> EasyEDA:R1206; symbol EasyEDA:RS-03K1583FT -> EasyEDA:CL1206FN158KPS; LCSC Part C321734 -> C53283992; MPN RS-03K1583FT -> CL1206FN158KPS; Manufacturer FH(风华) -> 昶龙科技
- R21, R22: value 0402WGF1003TCE -> FRC1206J104 TS; footprint EasyEDA:R0402 -> EasyEDA:R1206; symbol EasyEDA:0402WGF1003TCE -> EasyEDA:FRC1206J104TS; LCSC Part C25741 -> C2907421; MPN 0402WGF1003TCE -> FRC1206J104 TS; Manufacturer UNI-ROYAL(厚声) -> FOJAN(富捷)
- R33, R38: value AR02BTC1002 -> 1206W4F1002T5E; footprint EasyEDA:R0402 -> EasyEDA:R1206; symbol EasyEDA:AR02BTC1002 -> EasyEDA:1206W4F1002T5E; LCSC Part C317926 -> C17902; MPN AR02BTC1002 -> 1206W4F1002T5E; Manufacturer Viking(光颉) -> UNI-ROYAL(厚声)
- R9: value RC0603JR-071KL -> FRC1206F1R30TS; footprint EasyEDA:R0603 -> EasyEDA:R1206; symbol EasyEDA:RC0603JR-071KL -> EasyEDA:FRC1206F1R30TS; LCSC Part C14676 -> C2907365; MPN RC0603JR-071KL -> FRC1206F1R30TS; Manufacturer YAGEO(国巨) -> FOJAN(富捷)
Connections:
- net 3v is gone; now on net cs: SD_card_254.7
- net 5V is gone; now on net CD: SD_card_254.8
- net ESP32_enable is gone; now on net ESP32_enable_RJ12: R33.2, U9.6 (VO)
- net GND is gone; now on net DI: SD_card_254.6
- net +3V3: now also C29.1, J1.1, J1.2, SD_card_254.2, C11.1, C12.2; no longer C29.2
- net +5V: now also C19.1, C24.2, C25.2, C28.2; no longer C19.2, C24.1, C25.1, C28.1
- net CD: now also J1.7; no longer SD_card_254.1
- net CLK: now also J1.18, SD_card_254.4; no longer SD_card_254.5
- net DI: now also J1.17; no longer SD_card_254.3
- net DO: now also J1.19, SD_card_254.5; no longer SD_card_254.4
- net ESP32_FLT_Efuse: now also J1.6
- net ESP32_TX: now also J3.2
- net GND1: now also C19.2, C24.1, C25.1, C28.1, C29.2, J2.2, J3.1, J4.1, J4.2, SD_card_254.3, C11.2, C12.1; no longer C19.1, C24.2, C25.2, C28.2, C29.1
- net GPIO4_Battery: now also J1.4
- net cs: now also J1.20; no longer SD_card_254.2
- net 5V_ESP_module: now reaches J2.1
- net ESP32_enable_RJ12: now reaches J1.5
- no-connect marks 15 -> 4
Other:
- moved on the sheet: C29, C30, J1, J2, J3, J4, SD_card_254, U14, U15
