File: my_design/Slimme_meter_Sim -big-modular/Slimme_meter_Sim.kicad_pcb (KiCad board)
At the start: 2 copper layers, 123 x 181.8 mm, 129 parts, among them CN1 S2B-PH-SM4-TB, CN2 S2B-PH-SM4-TB, SW1 MSK12C02, SW2 TS665CJ, SW3 TS665CJ, SW4 SK-1500-L1?, U1 USBLC6-2SC6-ES, U10 6N137S_C20612601, U11 C1206C105K3RACAUTO, U12 C1206C105K3RACAUTO, U13 C1206C105K3RACAUTO, U2 BQ25185DLHR, U3 TPS61023DRLR, U4 TPS26625DRCR, U5 C1206C105K3RACAUTO, U6 SY8088AAC, U7 ESP32-C3-MINI-1-H4X, U8 6N137S_C20612601, U9 6N137S_C20612601

Commit message: Lock big-modular plan on DevKitC WROOM-2 with dual eFuse and safe 5V powering.
Document diode/switch power rules, USB-C/SD breakouts, N32R16V MCU module, and continue KiCad power sheets for the hand-build carrier.

Co-authored-by: Cursor <cursoragent@cursor.com>
Parts:
- added J1: PINHD_1x20_Female, Connector_PinSocket_2.54mm:PinSocket_1x20_P2.54mm_Vertical, F.Cu at (240.2, 166.0)
- added J2: PINHD_1x2_Female, Connector_PinSocket_2.54mm:PinSocket_1x02_P2.54mm_Vertical, F.Cu at (240.2, 216.8)
- added J3: PINHD_1x20_Female, Connector_PinSocket_2.54mm:PinSocket_1x20_P2.54mm_Vertical, F.Cu at (263.1, 166.0)
- added J4: PINHD_1x2_Female, Connector_PinSocket_2.54mm:PinSocket_1x02_P2.54mm_Vertical, F.Cu at (263.1, 216.8)
- added SD_card_254: PINHD_1x8_Female, Connector_PinSocket_2.54mm:PinSocket_1x08_P2.54mm_Vertical, F.Cu at (252.5, 96.5)
- added U14: TPS2553DBVR, EasyEDA:SOT-23-6_L2.9-W1.6-P0.95-LS2.8-BR, F.Cu at (226.7, 138.8)
- added U15: ESP32-S3-DevKitC, PCM_Espressif:ESP32-S3-DevKitC, F.Cu at (280.8, 162.5)
- added USB_c1: PINHD_1x6_Female, Connector_PinSocket_2.54mm:PinSocket_1x06_P2.54mm_Vertical, F.Cu at (292.1, 104.1)

Commit message: Checkpoint big-modular KiCad and FP6276B tooling before deeper power modularization.
Save DevKitC reference assets, USB-C breakout zip, boost datasheet/designer, and current schematic/PCB/library progress on the hand-build path.

Co-authored-by: Cursor <cursoragent@cursor.com>
Parts:
- removed 3v3: RH-5117, EasyEDA:TESTPOINT-TH_BD3.2-D1.6
- removed C13, C14, C16, C27: FS31X226M160EPG, EasyEDA:C1206
- removed C15, C18: CL05B104KO5NNNC, EasyEDA:C0402
- removed C17: CL05A105KA5NQNC, EasyEDA:C0402
- removed Card1: DM3AT-SF-PEJM5, EasyEDA:SD-SMD_DM3AT-SF-PEJM5
- removed D4: B5819W_C8598, EasyEDA:SOD-123_L2.7-W1.6-LS3.7-RD-1
- removed D5: RCLAMP0524P_C907837, EasyEDA:DFN2510-10_L2.5-W1.0-P0.50-BL
- removed GND1: RH-5002, EasyEDA:TESTPOINT-TH_BD2.5-D1.2_RH-5002
- removed L2: MDTA32251B-2R2M, EasyEDA:IND-SMD_L3.2-W2.5-BRL3225T100M
- removed LED3: DY-S505016/RGBC/6812F-NL-1T, EasyEDA:LED-SMD_4P-L5.0-W5.0-BR
- removed R1, R2: AR02BTC5101, EasyEDA:R0402
- removed R23: RT0402FRE07309RL, EasyEDA:R0402
- removed R24: SCR0402F68R1, EasyEDA:R0402
- removed R25, R26, R27, R29, R32, R34, R35, R36, R41, R42, R43, R44, R45, R46: AR02BTC1002, EasyEDA:R0402
- removed R28: 0402WGF3300TCE, EasyEDA:R0402
- removed SW2, SW3: TS665CJ, EasyEDA:SW-TH_4P-L6.0-W6.0-P4.50-LS6.5
- removed U1: USBLC6-2SC6-ES, EasyEDA:SOT-23-6_L2.9-W1.6-P0.95-LS2.8-BR
- removed U6: SY8088AAC, EasyEDA:SOT-23-5_L3.0-W1.7-P0.95-LS2.8-BR
- removed U7: ESP32-C3-MINI-1-H4X, EasyEDA:WIFIM-SMD_ESP32-C3-MINI-1
- removed USBC1: TYPE-C-31-M-12, foot:USB-C_SMD-TYPE-C-31-M-12_1
- removed USB_c1: PINHD_1x6_Female, Connector_PinSocket_2.54mm:PinSocket_1x06_P2.54mm_Vertical
- added J5: PINHD_1x8_Female, Connector_PinSocket_2.54mm:PinSocket_1x08_P2.54mm_Vertical, F.Cu at (69.3, 223.2)
- C11: value FS31X226M160EPG -> TCC1206M3L104J500FT
- C12: value CL05A105KA5NQNC -> FS31X226M160EPG; footprint EasyEDA:C0402 -> EasyEDA:C1206
- C19, C20, C21, C23, C24, C25, C28, C29, C31: value CL05B104KO5NNNC -> TCC1206M3L104J500FT; footprint EasyEDA:C0402 -> EasyEDA:C1206
- C8: value GRM188R71H223KA01D -> GRM3195C1H223JA01D; footprint EasyEDA:C0603 -> EasyEDA:C1206
- R10, R12, R21, R22, R39, R40: value 0402WGF1003TCE -> FRC1206J104 TS; footprint EasyEDA:R0402 -> EasyEDA:R1206
- R33, R38, R5: value AR02BTC1002 -> 1206W4F1002T5E; footprint EasyEDA:R0402 -> EasyEDA:R1206
- moved SD_card_254 161.5 mm to (152.3, 223.2)
- moved J1 137.8 mm to (106.0, 197.3)
- moved J2 137.8 mm to (106.0, 248.1)
- moved J3 137.8 mm to (128.9, 197.3)
- moved J4 137.8 mm to (128.9, 248.1)
- moved C11 117.6 mm to (221.4, 215.3)
- moved C12 117.6 mm to (221.8, 212.1)
- moved U14 38.5 mm to (203.6, 169.7)
- moved R39 18.6 mm to (139.1, 245.1)
- moved R40 18.6 mm to (139.1, 246.5)
- moved C31 18.6 mm to (139.0, 248.0)
- moved C29 17.7 mm to (146.9, 228.8), turned to 180 degrees
- moved R38 15.3 mm to (99.9, 237.7)
- moved C30 14.1 mm to (146.9, 231.8)
- moved C20 7.74 mm to (77.0, 210.3), turned to 90 degrees
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Connections:
- BT1 pad 1: GND1 -> GND
- Batt_power_on_SW1 pad 4: GND1 -> GND
- C1 pad 1: GND1 -> GND
- C10 pad 1: GND1 -> GND
- C11 pad 1: GND1 -> 3v
- C11 pad 2: +3V3 -> GND
- C12 pad 1: GND1 -> GND
- C12 pad 2: Net-(U6-EN) -> 3v
- C19 pad 1: GND1 -> +5V
- C19 pad 2: +5V -> GND
- C2 pad 1: GND1 -> GND
- C20 pad 1: GND1 -> Net-(D1-C)
- C20 pad 2: Net-(D1-C) -> GND
- C21 pad 1: VCC -> GND
- C21 pad 2: GND1 -> VCC
- C22 pad 2: GND1 -> GND
- C23 pad 1: +5V -> GND
- C23 pad 2: GND1 -> +5V
- C24 pad 1: +5V -> GND
- C24 pad 2: GND1 -> +5V
- C25 pad 1: +5V -> GND
- C25 pad 2: GND1 -> +5V
- C28 pad 1: +5V -> GND
- C28 pad 2: GND1 -> +5V
- C29 pad 1: GND1 -> 3v
- C29 pad 2: +3V3 -> GND
- C3 pad 1: GND1 -> GND
- C30 pad 1: GND1 -> GND
- C30 pad 2: +3V3 -> 3v
- C31 pad 1: /SCH_1_USB_5volt/GPIO4_Battery -> GND
- C31 pad 2: GND1 -> /SCH_1_USB_5volt/GPIO4_Battery
- C4 pad 2: GND1 -> GND
- C5 pad 2: GND1 -> GND
- C6 pad 2: GND1 -> GND
- C7 pad 1: GND1 -> GND
- C9 pad 1: GND1 -> GND
- CN1 pad 2: GND1 -> GND
- CN1 pad 3: GND1 -> GND
- CN1 pad 4: GND1 -> GND
- CN2 pad 2: GND1 -> GND
- CN2 pad 3: GND1 -> GND
- CN2 pad 4: GND1 -> GND
- D2 pad 2: GND1 -> GND
- D3 pad 2: GND1 -> GND
- J1 pad 1: unconnected-(J1-Pad1) -> 3v
- J1 pad 17: unconnected-(J1-Pad17) -> DI
- J1 pad 18: unconnected-(J1-Pad18) -> CLK
- J1 pad 19: unconnected-(J1-Pad19) -> DO
- J1 pad 2: unconnected-(J1-Pad2) -> 3v
- J1 pad 20: unconnected-(J1-Pad20) -> cs
- J1 pad 4: unconnected-(J1-Pad4) -> /SCH_1_USB_5volt/GPIO4_Battery
- J1 pad 5: unconnected-(J1-Pad5) -> /SCH_2_power_supplies/ESP32_enable_RJ12
- J1 pad 6: unconnected-(J1-Pad6) -> /SCH_2_power_supplies/ESP32_FLT_Efuse
- J1 pad 7: unconnected-(J1-Pad7) -> CD
- J2 pad 1: unconnected-(J2-Pad1) -> /SCH_2_power_supplies/5V_ESP_module
- J2 pad 2: unconnected-(J2-Pad2) -> GND
- J3 pad 1: unconnected-(J3-Pad1) -> GND
- J3 pad 2: unconnected-(J3-Pad2) -> /SCH_2_power_supplies/ESP32_TX
- J4 pad 1: unconnected-(J4-Pad1) -> GND
- J4 pad 2: unconnected-(J4-Pad2) -> GND
- LED1 pad 1: GND1 -> GND
- LED2 pad 1: GND1 -> GND
- R12 pad 1: GND1 -> GND
- R33 pad 1: +3V3 -> 3v
- R33 pad 2: /SCH_2_power_supplies/ESP32_enable -> /SCH_2_power_supplies/ESP32_enable_RJ12
- R38 pad 1: +3V3 -> 3v
- R40 pad 2: GND1 -> GND
- R5 pad 1: GND1 -> GND
- R6 pad 1: GND1 -> GND
- R7 pad 1: GND1 -> GND
- RJ1 pad 3: GND1 -> GND
- RJ1 pad 6: GND1 -> GND
- SD_card_254 pad 1: CD -> unconnected-(SD_card_254-Pad1)
- SD_card_254 pad 2: cs -> 3v
- SD_card_254 pad 3: DI -> GND
- SD_card_254 pad 4: DO -> CLK
- SD_card_254 pad 5: CLK -> DO
- SD_card_254 pad 6: GND -> DI
- SD_card_254 pad 7: 3v -> cs
- SD_card_254 pad 8: 5V -> CD
- SW1 pad 1: GND1 -> GND
- SW1 pad 4: GND1 -> GND
- SW4 pad 10: GND1 -> GND
- SW4 pad 7: GND1 -> GND
- SW4 pad 8: GND1 -> GND
- SW4 pad 9: GND1 -> GND
- TP3 pad 1: GND1 -> GND
- U10 pad 1: GND1 -> GND
- U10 pad 4: GND1 -> GND
- U10 pad 5: GND1 -> GND
- U11 pad 2: GND1 -> GND
- U12 pad 2: GND1 -> GND
- U13 pad 2: GND1 -> GND
- U2 pad 11: GND1 -> GND
- U2 pad 4: GND1 -> GND
- U2 pad 5: GND1 -> GND
- U3 pad 4: GND1 -> GND
- U4 pad 11: GND1 -> GND
- U4 pad 6: GND1 -> GND
- U5 pad 1: GND1 -> GND
- U8 pad 1: GND1 -> GND
- U8 pad 3: GND1 -> GND
- U8 pad 4: GND1 -> GND
- U8 pad 5: GND1 -> GND
- U9 pad 1: GND1 -> GND
- U9 pad 3: GND1 -> GND
- U9 pad 4: GND1 -> GND
- U9 pad 5: GND1 -> GND
- U9 pad 6: /SCH_2_power_supplies/ESP32_enable -> /SCH_2_power_supplies/ESP32_enable_RJ12
- USB_power_on_SW1 pad 4: GND1 -> GND
Routing:
- net +3V3: track 231.0 -> 0.00 mm, vias 4 -> 0
- net +5V: track 262.7 -> 111.2 mm, vias 15 -> 9
- net VBATT: track 107.6 -> 0.00 mm, vias 6 -> 0
- net VCC: track 94.4 -> 10.4 mm, vias 34 -> 10
- net /SCH_2_power_supplies/ESP32_TX: track 73.2 -> 0.00 mm, vias 2 -> 0
- net /SCH_2_power_supplies/SD_CD_SW_A: track 67.7 -> 0.00 mm, vias 2 -> 0
- net /SCH_2_power_supplies/GPIO6_CS: track 61.5 -> 0.00 mm, vias 4 -> 0
- net /SCH_2_power_supplies/ESP32_enable: track 58.3 -> 0.00 mm, vias 2 -> 0
- net /SCH_2_power_supplies/ESP32_FLT_Efuse: track 50.6 -> 0.00 mm, vias 2 -> 0
- net /SCH_2_power_supplies/GPIO1_MOSI_CMD: track 48.1 -> 0.00 mm, vias 2 -> 0
- net /SCH_2_power_supplies/GPIO0_SCK: track 47.9 -> 0.00 mm, vias 4 -> 0
- net USB_D-: track 44.1 -> 0.00 mm
- net USB_D+: track 44.1 -> 0.00 mm
- net /SCH_2_power_supplies/GPIO3_MISO: track 43.5 -> 0.00 mm, vias 2 -> 0
- net /SCH_2_power_supplies/RJ12_Tx_pin5: track 42.2 -> 0.00 mm
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- removed copper zone on B.Cu, net GND1
- removed copper zone on F.Cu, net GND1
- removed copper zone on F.Cu, net Net-(D1-C)
- removed copper zone on B.Cu, net VBATT
- removed copper zone on F.Cu, net VBATT
- removed copper zone on B.Cu, net VCC
Other:
- board size 123 x 181.8 mm -> 128.9 x 183.6 mm
- board text removed: "BOOT"
- board text removed: "Restart"
